File: pcb/plaid.kicad_pcb (KiCad board)
At the start: 2 copper layers, 228 x 98 mm, 139 parts, among them J1 USB_OTG, J2 AVR_ISP_6, J3 Conn_01x04, J4 GS2, J5 GS2, SW1 SW_Push, SW10 SW_Push, SW11 SW_Push, SW12 SW_Push, SW13 SW_Push, SW14 SW_Push, SW15 SW_Push, SW16 SW_Push, SW17 SW_Push, SW18 SW_Push, SW19 SW_Push, SW2 SW_Push, SW20 SW_Push, SW21 SW_Push, SW22 SW_Push, SW23 SW_Push, SW24 SW_Push, SW25 SW_Push, SW26 SW_Push, SW27 SW_Push, SW28 SW_Push, SW29 SW_Push, SW3 SW_Push, SW30 SW_Push, SW31 SW_Push, SW32 SW_Push, SW33 SW_Push, SW34 SW_Push, SW35 SW_Push, SW36 SW_Push, SW37 SW_Push, SW38 SW_Push, SW39 SW_Push, SW4 SW_Push, SW40 SW_Push, SW41 SW_Push, SW42 SW_Push, SW43 SW_Push, SW44 SW_Push, SW45 SW_Push, SW46 SW_Push, SW47 SW_Push, SW48 SW_Push, SW49 SW_Push, SW5 SW_Push, SW50 RESET, SW51 BOOT, SW6 SW_Push, SW7 SW_Push, SW8 SW_Push, SW9 SW_Push, U1 ATMEGA328-PU, Y1 16MHz

Commit message: Switch to USB-C
Parts:
- removed D49, D50: 3.6V, dm9_rc:D_DO-35_SOD27_P5.08mm_Horizontal
- removed F1: 100mA, dm9_miscs:polyfuse_5.1mm
- removed G***: LOGO, plaid_silk:plaid_silk
- removed G***: LOGO, dm9_silks:logo_hsgw_7_5mm
- removed G***: LOGO, dm9_silks:logo_dm9_15mm
- removed G***: LOGO, plaid_silk:plaid_katakana
- removed J1: USB_OTG, dm9_conn:USB_MINIB_Akizuki_MUSB-5BF01AS
- removed J3: Conn_01x04, Pin_Headers:Pin_Header_Straight_1x04_Pitch2.54mm
- removed J4, J5: GS2, Connectors:GS2
- removed LED1: RED, LEDs:LED_D3.0mm
- removed LED2: GREEN, LEDs:LED_D3.0mm
- removed R1, R7, R8: 1.5k, Resistors_THT:R_Axial_DIN0204_L3.6mm_D1.6mm_P5.08mm_Horizontal
- removed R2, R3: 75R, Resistors_THT:R_Axial_DIN0204_L3.6mm_D1.6mm_P5.08mm_Horizontal
- removed R5, R6: I2C, Resistors_THT:R_Axial_DIN0204_L3.6mm_D1.6mm_P5.08mm_Horizontal
- removed REF**: Stab_MX_2u, SMKJP:Stab_MX_2u
- added D51: 3.6V, cftkb:D_DO-35_SOD27_P5.08mm_Horizontal, F.Cu at (241.3, 59.0)
- added D52: 3.6V, cftkb:D_DO-35_SOD27_P5.08mm_Horizontal, F.Cu at (238.5, 59.0)
- added F2: 500mA, cftkb:polyfuse_5.1mm, F.Cu at (250.9, 67.1)
- added R10: 5.1k, Resistor_THT:R_Axial_DIN0204_L3.6mm_D1.6mm_P5.08mm_Horizontal, F.Cu at (262.2, 61.4)
- added R11: 5.1k, Resistor_THT:R_Axial_DIN0204_L3.6mm_D1.6mm_P5.08mm_Horizontal, F.Cu at (257.1, 59.1)
- added R12: 75R, Resistor_THT:R_Axial_DIN0204_L3.6mm_D1.6mm_P5.08mm_Horizontal, F.Cu at (231.0, 55.4)
- added R13: 75R, Resistor_THT:R_Axial_DIN0204_L3.6mm_D1.6mm_P5.08mm_Horizontal, F.Cu at (231.0, 57.7)
- added R9: 1.5k, Resistor_THT:R_Axial_DIN0204_L3.6mm_D1.6mm_P5.08mm_Horizontal, F.Cu at (231.0, 53.1)
- added USB1: Type-C_USB_C_GCT_USB4085, cftkb:USB_C_GCT_USB4085, F.Cu at (249.5, 52.5)
- C3: value 10u -> 4.7u
Connections:
- U1 pad 21: (no net) -> Net-(U1-Pad21)
Routing:
- net /i2c_SDA: track 56.9 -> 2.69 mm
- net /i2c_SCL: track 46.3 -> 0.00 mm
- net +5V: track 127.6 -> 91.2 mm
- net Net-(D51-Pad1): track 0.00 -> 33.4 mm, vias 0 -> 1
- net Net-(D52-Pad1): track 0.00 -> 33.2 mm, vias 0 -> 1
- net GND: track 8.83 -> 36.7 mm, vias 79 -> 76
- net Net-(D50-Pad1): track 18.9 -> 0.00 mm
- net Net-(R11-Pad1): track 0.00 -> 16.8 mm
- net Net-(D49-Pad1): track 15.6 -> 0.00 mm
- net VCC: track 0.00 -> 14.5 mm
- net Net-(R10-Pad2): track 0.00 -> 9.72 mm, vias 0 -> 1
- net Net-(LED1-Pad2): track 9.46 -> 0.00 mm
- net Net-(LED2-Pad2): track 8.56 -> 0.00 mm
- net Net-(J5-Pad1): track 6.87 -> 0.00 mm
- net Net-(J4-Pad1): track 6.35 -> 0.00 mm
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Other:
- net class Default: clearance 0.3 -> 0.2; trace_width 0.3 -> 0.254
- rule pad_to_mask_clearance: 0.2 -> 0.051
- rule solder_mask_min_width: 0.2 -> 0.25
- rule trace_clearance: 0.3 -> 0.2
- board text removed: "5V"
- board text removed: "GND"
- board text removed: "LED"
- board text removed: "SCL"
- board text removed: "SDA"
