File: pcb/plaid.sch (KiCad schematic (older format))
At the start: 127 parts, among them J2 AVR_ISP_6, SW1 SW_Push, SW10 SW_Push, SW11 SW_Push, SW12 SW_Push, SW13 SW_Push, SW14 SW_Push, SW15 SW_Push, SW16 SW_Push, SW17 SW_Push, SW18 SW_Push, SW19 SW_Push, SW2 SW_Push, SW20 SW_Push, SW21 SW_Push, SW22 SW_Push, SW23 SW_Push, SW24 SW_Push, SW25 SW_Push, SW26 SW_Push, SW27 SW_Push, SW28 SW_Push, SW29 SW_Push, SW3 SW_Push, SW30 SW_Push, SW31 SW_Push, SW32 SW_Push, SW33 SW_Push, SW34 SW_Push, SW35 SW_Push, SW36 SW_Push, SW37 SW_Push, SW38 SW_Push, SW39 SW_Push, SW4 SW_Push, SW40 SW_Push, SW41 SW_Push, SW42 SW_Push, SW43 SW_Push, SW44 SW_Push, SW45 SW_Push, SW46 SW_Push, SW47 SW_Push, SW48 SW_Push, SW49 SW_Push, SW5 SW_Push, SW50 RESET, SW51 BOOT, SW6 SW_Push, SW7 SW_Push, SW8 SW_Push, SW9 SW_Push, U1 ATMEGA328-PU, Y1 16MHz

Commit message: RGB LED setup
Parts:
- added C6: 100n, Capacitor_THT:C_Disc_D4.3mm_W1.9mm_P5.00mm, symbol Device:C_Small
- added D49: SK6812, LED_SMD:LED_SK6812_PLCC4_5.0x5.0mm_P3.2mm, symbol LED:SK6812
Connections:
- net labels added: RGB_LED
- net labels removed: i2c_SCL, i2c_SDA
- wire segments 252 -> 257
- no-connect marks 3 -> 4
Changed lines of the file:
@@
 $EndComp
 NoConn ~ 1800 4500
-Text Label 3100 5800 0    50   ~ 0
-i2c_SDA
 Wire Wire Line
 	4300 6700 4300 6800
-Text Label 3100 5900 0    50   ~ 0
-i2c_SCL
 Wire Wire Line
 	3000 6600 3100 6600
@@
 Wire Wire Line
 	3050 1800 3150 1800
+$Comp
+L LED:SK6812 D49
+U 1 1 5E125DCB
+P 5350 6150
+F 0 "D49" H 5694 6196 50  0000 L CNN
+F 1 "SK6812" H 5694 6105 50  0000 L CNN
+F 2 "LED_SMD:LED_SK6812_PLCC4_5.0x5.0mm_P3.2mm" H 5400 5850 50  0001 L TNN
+F 3 "https://cdn-shop.adafruit.com/product-files/1138/SK6812+LED+datasheet+.pdf" H 5450 5775 50  0001 L TNN
+	1    5350 6150
+	1    0    0    -1
+$EndComp
+NoConn ~ 5650 6150
+Text Label 3100 5800 0    50   ~ 0
+RGB_LED
+Text Label 4700 6150 0    50   ~ 0
+RGB_LED
+Wire Wire Line
+	4700 6150 5050 6150
+$Comp
+L power:GND #PWR0102
+U 1 1 5E19A614
+P 5350 6450
+F 0 "#PWR0102" H 5350 6200 50  0001 C CNN
+F 1 "GND" H 5355 6277 50  0000 C CNN
+F 2 "" H 5350 6450 50  0001 C CNN
+F 3 "" H 5350 6450 50  0001 C CNN
+	1    5350 6450
+	1    0    0    -1
+$EndComp
+$Comp
+L power:+5V #PWR0103
+U 1 1 5E19BA47
+P 5350 5750
+F 0 "#PWR0103" H 5350 5600 50  0001 C CNN
+F 1 "+5V" H 5365 5923 50  0000 C CNN
+F 2 "" H 5350 5750 50  0001 C CNN
+F 3 "" H 5350 5750 50  0001 C CNN
+	1    5350 5750
+	1    0    0    -1
+$EndComp
+$Comp
+L Device:C_Small C6
+U 1 1 5E1CE4B8
+P 6150 5950
+F 0 "C6" H 6242 5996 50  0000 L CNN
+F 1 "100n" H 6242 5905 50  0000 L CNN
+F 2 "Capacitor_THT:C_Disc_D4.3mm_W1.9mm_P5.00mm" H 6150 5950 50  0001 C CNN
+F 3 "~" H 6150 5950 50  0001 C CNN
+	1    6150 5950
+	-1   0    0    1
+$EndComp
+Wire Wire Line
+	5350 5750 5350 5800
+Connection ~ 5350 5800
+Wire Wire Line
+	5350 5800 5350 5850
+Wire Wire Line
+	6150 5800 6150 5850
+Wire Wire Line
+	5350 5800 6150 5800
+$Comp
+L power:GND #PWR01
+U 1 1 5E263524
+P 6150 6050
+F 0 "#PWR01" H 6150 5800 50  0001 C CNN
+F 1 "GND" H 6155 5877 50  0000 C CNN
+F 2 "" H 6150 6050 50  0001 C CNN
+F 3 "" H 6150 6050 50  0001 C CNN
+	1    6150 6050
+	1    0    0    -1
+$EndComp
 $EndSCHEMATC

Commit message: Add usb-c, rgb led
Parts:
- removed D47, D48: 1N4148, dm9_rc:D_DO-35_SOD27_P5.08mm_Horizontal, symbol Device:D_Small_ALT
- removed SW47, SW48: SW_Push, SMKJP:SW_Cherry_MX1A_1.00u_PCB, symbol Switch:SW_Push
- removed SW49: SW_Push, SMKJP:SW_Cherry_MX1A_2.0U_PCB_universal_center, symbol Switch:SW_Push
- SW41, SW42: footprint SMKJP:SW_Cherry_MX1A_1.00u_PCB -> cftkb:SW_Cherry_MX1A_2.00u_PCBNOSCREEN
Connections:
- wire segments 257 -> 248
Changed lines of the file:
@@
 F 0 "SW41" H 7200 3785 50  0000 C CNN
 F 1 "SW_Push" H 7200 3694 50  0000 C CNN
-F 2 "SMKJP:SW_Cherry_MX1A_1.00u_PCB" H 7200 3700 50  0001 C CNN
+F 2 "cftkb:SW_Cherry_MX1A_2.00u_PCBNOSCREEN" H 7200 3700 50  0001 C CNN
 F 3 "" H 7200 3700 50  0001 C CNN
 	1    7200 3500
@@
 L Switch:SW_Push SW42
 U 1 1 5C149FBD
-P 7700 4200
-F 0 "SW42" H 7700 4485 50  0000 C CNN
-F 1 "SW_Push" H 7700 4394 50  0000 C CNN
-F 2 "SMKJP:SW_Cherry_MX1A_1.00u_PCB" H 7700 4400 50  0001 C CNN
-F 3 "" H 7700 4400 50  0001 C CNN
-	1    7700 4200
+P 7700 3500
+F 0 "SW42" H 7700 3785 50  0000 C CNN
+F 1 "SW_Push" H 7700 3694 50  0000 C CNN
+F 2 "cftkb:SW_Cherry_MX1A_2.00u_PCBNOSCREEN" H 7700 3700 50  0001 C CNN
+F 3 "" H 7700 3700 50  0001 C CNN
+	1    7700 3500
 	-1   0    0    -1
 $EndComp
@@
 L Device:D_Small_ALT D42
 U 1 1 5C149FC3
-P 7900 4000
-F 0 "D42" V 7900 3750 50  0000 L CNN
-F 1 "1N4148" V 8000 3600 50  0000 L CNN
-F 2 "dm9_rc:D_DO-35_SOD27_P5.08mm_Horizontal" V 7900 4000 50  0001 C CNN
-F 3 "~" V 7900 4000 50  0001 C CNN
-	1    7900 4000
-	0    -1   1    0
+P 7900 3700
+F 0 "D42" V 7900 3450 50  0000 L CNN
+F 1 "1N4148" V 8000 3300 50  0000 L CNN
+F 2 "dm9_rc:D_DO-35_SOD27_P5.08mm_Horizontal" V 7900 3700 50  0001 C CNN
+F 3 "~" V 7900 3700 50  0001 C CNN
+	1    7900 3700
+	0    1    -1   0
 $EndComp
 Connection ~ 7500 1400
@@
 Wire Wire Line
 	10400 2800 10400 2900
-$Comp
-L Switch:SW_Push SW47
-U 1 1 5C14C2A4
-P 10200 3500
-F 0 "SW47" H 10200 3785 50  0000 C CNN
-F 1 "SW_Push" H 10200 3694 50  0000 C CNN
-F 2 "SMKJP:SW_Cherry_MX1A_1.00u_PCB" H 10200 3700 50  0001 C CNN
-F 3 "" H 10200 3700 50  0001 C CNN
-	1    10200 3500
-	-1   0    0    -1
-$EndComp
-$Comp
-L Device:D_Small_ALT D47
-U 1 1 5C14C2AA
-P 10400 3700
-F 0 "D47" V 10450 3550 50  0000 L CNN
-F 1 "1N4148" V 10350 3350 50  0000 L CNN
-F 2 "dm9_rc:D_DO-35_SOD27_P5.08mm_Horizontal" V 10400 3700 50  0001 C CNN
-F 3 "~" V 10400 3700 50  0001 C CNN
-	1    10400 3700
-	0    1    -1   0
-$EndComp
-Wire Wire Line
-	10400 3500 10400 3600
-Wire Wire Line
-	10000 3500 10000 2800
 Connection ~ 10000 1400
 Wire Wire Line
@@
 Wire Wire Line
 	10000 2100 10000 1400
-Connection ~ 10000 2800
 Wire Wire Line
 	10000 2800 10000 2100
@@
 Wire Wire Line
 	10900 2800 10900 2900
-$Comp
-L Switch:SW_Push SW48
-U 1 1 5C14C2E3
-P 10700 3500
-F 0 "SW48" H 10700 3785 50  0000 C CNN
-F 1 "SW_Push" H 10700 3694 50  0000 C CNN
-F 2 "SMKJP:SW_Cherry_MX1A_1.00u_PCB" H 10700 3700 50  0001 C CNN
-F 3 "" H 10700 3700 50  0001 C CNN
-	1    10700 3500
-	-1   0    0    -1
-$EndComp
-$Comp
-L Device:D_Small_ALT D48
-U 1 1 5C14C2E9
-P 10900 3700
-F 0 "D48" V 10950 3550 50  0000 L CNN
-F 1 "1N4148" V 10850 3350 50  0000 L CNN
-F 2 "dm9_rc:D_DO-35_SOD27_P5.08mm_Horizontal" V 10900 3700 50  0001 C CNN
-F 3 "~" V 10900 3700 50  0001 C CNN
-	1    10900 3700
-	0    1    -1   0
-$EndComp
-Wire Wire Line
-	10900 3500 10900 3600
-Wire Wire Line
-	10500 3500 10500 2800
 Connection ~ 10500 1400
 Wire Wire Line
@@
 Wire Wire Line
 	10500 2100 10500 1400
-Connection ~ 10500 2800
 Wire Wire Line
 	10500 2800 10500 2100
@@
 Wire Wire Line
 	4700 5100 4900 5100
-$Comp
-L Switch:SW_Push SW49
-U 1 1 5C089CEA
-P 7700 4600
-F 0 "SW49" H 7700 4885 50  0000 C CNN
-F 1 "SW_Push" H 7700 4794 50  0000 C CNN
-F 2 "SMKJP:SW_Cherry_MX1A_2.0U_PCB_universal_center" H 7700 4800 50  0001 C CNN
-F 3 "" H 7700 4800 50  0001 C CNN
-	1    7700 4600
-	-1   0    0    -1
-$EndComp
-Wire Wire Line
-	7900 3900 7900 3800
-Wire Wire Line
-	7900 4100 7900 4200
-Connection ~ 7500 4200
-Wire Wire Line
-	7500 4200 7500 4600
-Connection ~ 7900 4200
-Wire Wire Line
-	7900 4200 7900 4600
-Wire Wire Line
-	7500 2800 7500 4200
+Wire Wire Line
+	7900 3600 7900 3500
+Wire Wire Line
+	7500 2800 7500 3500
 $Comp
 L Mechanical:MountingHole H3
@@
 Wire Wire Line
 	9400 3800 9900 3800
-Connection ~ 9900 3800
-Wire Wire Line
-	9900 3800 10400 3800
-Connection ~ 10400 3800
-Wire Wire Line
-	10400 3800 10900 3800
 Wire Wire Line
 	1900 1400 2050 1400
